Commit message: Add files via upload

File: src/amr_description/urdf/amr_description.urdf (robot description, URDF)
Before this commit: robot amr_description, 14 links, 13 joints
Links:
- removed link rear_caster_stear_left_link
- removed link rear_caster_stear_right_link
- added link rear_caster_steer_left_link, mass 0.0164104146999673; collision mesh filename=package://amr_description/meshes/rear_caster_steer_left_lin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; visual mesh filename=package://amr_description/meshes/rear_caster_steer_left_lin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
- added link rear_caster_steer_right_link, mass 0.0179822997869202; collision mesh filename=package://amr_description/meshes/rear_caster_steer_right_li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; visual mesh filename=package://amr_description/meshes/rear_caster_steer_right_li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
- link base_lift_link: mass 0.30532 -> 0.326486799501112
- link base_link: mass 2.5717 -> 4.30533644141521
- link camera_link: mass 0.22579 -> 0.183480710290439
- link encoder_lift_link: mass 0.34037 -> 0.357360840342875
- link front_encoder_wheel_left_link: mass 0.024134 -> 0.0241340978121404
- link front_encoder_wheel_right_link: mass 0.024134 -> 0.0241340978121404
- link imu_link: mass 0.43383 -> 0.433591677658542
- link left_fork_link: mass 0.049955 -> 0.0680578875808647
- link lidar_link: mass 0.14165 -> 0.141654473640087
- link rear_caster_wheel_left_link: mass 0.029434 -> 0.0294337031863833
- link rear_caster_wheel_right_link: mass 0.029434 -> 0.0294337031863833
- link right_fork_link: mass 0.049955 -> 0.0680578875808845
Joints:
- removed joint left_fork_joint
- removed joint rear_caster_stear_left_joint
- removed joint rear_caster_stear_right_joint
- added joint left_fork_right: type fixed, parent encoder_lift_link, child left_fork_link, origin xyz=0.1275 0.086108 -0.042399 rpy=0 0 0, axis 0 0 0
- added joint rear_caster_steer_left_joint: type continuous, parent base_link, child rear_caster_steer_left_link, origin xyz=-0.20168 0.19842 -0.030503 rpy=0 0 0, axis 0 0 1
- added joint rear_caster_steer_right_joint: type continuous, parent base_link, child rear_caster_steer_right_link, origin xyz=-0.20168 -0.18778 -0.030503 rpy=0 0 0, axis 0 0 1
- joint camera_joint: origin xyz=0.091175 -0.17618 0.36182 rpy=0 0 0 -> xyz=0.10152 0.014743 0.59519 rpy=0 0 0
- joint encoder_lift_joint: limit lower=0 upper=0.87 effort=100 velocity=1.0 -> lower=-0.04 upper=0.85 effort=50 velocity=0.1
- joint lidar_joint: origin xyz=-0.034802 -0.0038905 0.10975 rpy=0 0 0 -> xyz=-0.024802 -0.0038905 0.12806 rpy=0 0 0
- joint rear_caster_wheel_left_joint: parent rear_caster_stear_left_link -> rear_caster_steer_left_link
- joint rear_caster_wheel_right_joint: parent rear_caster_stear_right_link -> rear_caster_steer_right_link
- joint right_fork_joint: limit lower=0 upper=0 effort=0 velocity=0 -> (none); origin xyz=0.1275 -0.085344 -0.093107 rpy=0 0 0 -> xyz=0.1275 -0.085344 -0.042399 rpy=0 0 0

Commit message: Update amr_description.urdf

File: src/amr_description/urdf/amr_description.urdf (robot description, URDF)
Before this commit: robot amr_description, 14 links, 13 joints
Links:
- link base_link: mass 4.30533644141521 -> 15.30533644141521
Joints:
- joint front_encoder_wheel_left_joint: limit (none) -> effort=0.863 velocity=11.52
- joint front_encoder_wheel_right_joint: limit (none) -> effort=0.863 velocity=11.52

Commit message: Update amr_description.urdf

File: src/amr_description/urdf/amr_description.urdf (robot description, URDF)
Before this commit: robot amr_description, 14 links, 13 joints
Links:
- link base_link: mass 15.30533644141521 -> 4.30533644141521

Commit message: Add files via upload

File: src/amr_description/urdf/amr_description.urdf (robot description, URDF)
Before this commit: robot amr_description, 14 links, 13 joints
Links:
- link base_lift_link: mass 0.326486799501112 -> 0.32649
- link base_link: mass 4.30533644141521 -> 4.3053
- link camera_link: mass 0.183480710290439 -> 0.18348
- link encoder_lift_link: mass 0.357360840342875 -> 0.35736
- link front_encoder_wheel_left_link: mass 0.0241340978121404 -> 0.024134
- link front_encoder_wheel_right_link: mass 0.0241340978121404 -> 0.024134
- link imu_link: mass 0.433591677658542 -> 0.43359
- link left_fork_link: mass 0.0680578875808647 -> 0.068058
- link lidar_link: mass 0.141654473640087 -> 0.14165
- link rear_caster_steer_left_link: mass 0.0164104146999673 -> 0.01641
- link rear_caster_steer_right_link: mass 0.0179822997869202 -> 0.017982
- link rear_caster_wheel_left_link: mass 0.0294337031863833 -> 0.029434
- link rear_caster_wheel_right_link: mass 0.0294337031863833 -> 0.029434
- link right_fork_link: mass 0.0680578875808845 -> 0.068058
Joints:
- joint base_lift_joint: origin xyz=0.12352 0.0055154 0.017997 rpy=0 0 0 -> xyz=0.192 0.00019696 0.020997 rpy=0 0 0
- joint camera_joint: origin xyz=0.10152 0.014743 0.59519 rpy=0 0 0 -> xyz=0.17 0.0094248 0.59819 rpy=0 0 0
- joint encoder_lift_joint: limit lower=-0.04 upper=0.85 effort=50 velocity=0.1 -> lower=-0.04 upper=0.8 effort=50 velocity=0.1
- joint front_encoder_wheel_left_joint: origin xyz=0.074022 0.24142 -0.063003 rpy=0 0 0 -> xyz=0.1425 0.2361 -0.060003 rpy=0 0 0
- joint front_encoder_wheel_right_joint: origin xyz=0.074022 -0.23078 -0.063003 rpy=0 0 0 -> xyz=0.1425 -0.2361 -0.060003 rpy=0 0 0
- joint imu_joint: origin xyz=0 0 0 rpy=0 0 0 -> xyz=0.068481 -0.0053185 0.003 rpy=0 0 0
- joint lidar_joint: origin xyz=-0.024802 -0.0038905 0.12806 rpy=0 0 0 -> xyz=0.043679 -0.0092089 0.13106 rpy=0 0 0
- joint rear_caster_steer_left_joint: origin xyz=-0.20168 0.19842 -0.030503 rpy=0 0 0 -> xyz=-0.1332 0.1931 -0.027503 rpy=0 0 0
- joint rear_caster_steer_right_joint: origin xyz=-0.20168 -0.18778 -0.030503 rpy=0 0 0 -> xyz=-0.1332 -0.1931 -0.027503 rpy=0 0 0
