Commit message: Add files via upload

File: amr_description/urdf/amr.gazebo.xacro (robot description, xacro)
@@ -19,11 +19,32 @@
   <gazebo reference="front_encoder_wheel_left_link">
     <material>Gazebo/Black</material>
-    <mu1>1.0</mu1>
-    <mu2>1.0</mu2>
+    <mu1>0.8</mu1>
+    <mu2>0.8</mu2>
+    <kp>1e8</kp>
+    <kd>100</kd>
   </gazebo>
   <gazebo reference="front_encoder_wheel_right_link">
     <material>Gazebo/Black</material>
-    <mu1>1.0</mu1>
-    <mu2>1.0</mu2>
+    <mu1>0.8</mu1>
+    <mu2>0.8</mu2>
+    <kp>1e8</kp>
+    <kd>100</kd>
+  </gazebo>
+  <!-- ============================================================ -->
+  <!-- CASTER WHEEL FRICTION (low friction for free rolling)        -->
+  <!-- ============================================================ -->
+  <gazebo reference="rear_caster_wheel_left_link">
+    <material>Gazebo/Grey</material>
+    <mu1>0.3</mu1>
+    <mu2>0.3</mu2>
+    <kp>1e6</kp>
+    <kd>10</kd>
+  </gazebo>
+  <gazebo reference="rear_caster_wheel_right_link">
+    <material>Gazebo/Grey</material>
+    <mu1>0.3</mu1>
+    <mu2>0.3</mu2>
+    <kp>1e6</kp>
+    <kd>10</kd>
   </gazebo>
   <!-- ============================================================ -->
@@ -33,5 +54,5 @@
     <sensor type="ray" name="lidar_sensor">
       <pose>0 0 0 0 0 0</pose>
-      <visualize>true</visualize>
+      <visualize>false</visualize>
       <update_rate>10</update_rate>
       <ray>

Commit message: Nav2 config

File: amr_description/urdf/amr.gazebo.xacro (robot description, xacro)
@@ -64,4 +64,6 @@
   <gazebo reference="encoder_lift_link">
     <material>Gazebo/White</material>
+    <mu1>0.2</mu1><mu2>0.2</mu2><kp>1e4</kp><kd>10.0</kd>
+    <minDepth>0.001</minDepth><maxVel>0.1</maxVel>
   </gazebo>
   <gazebo reference="left_fork_link">
@@ -172,5 +174,6 @@
         <namespace>/</namespace>
         <remapping>cmd_vel:=/diff_drive/cmd_vel</remapping>
-        <remapping>odom:=odom</remapping>
+        <!-- Đẩy dữ liệu thô vào /odom_raw -->
+        <remapping>odom:=/odom_raw</remapping>
       </ros>
       <!-- Drive wheels (front encoder wheels) -->
@@ -186,5 +189,5 @@
       <publish_odom>true</publish_odom>
       <publish_odom_tf>false</publish_odom_tf>
-      <publish_wheel_tf>false</publish_wheel_tf>
+      <publish_wheel_tf>true</publish_wheel_tf>
       <odometry_frame>odom</odometry_frame>
       <robot_base_frame>base_footprint</robot_base_frame>
@@ -202,8 +205,8 @@
         <remapping>~/out:=joint_states</remapping>
       </ros>
-      <update_rate>50</update_rate>  <!-- Reduced from 50 to match sim time -->
+      <update_rate>30</update_rate>  <!-- Reduced from 50 to match sim time -->
       <!-- Drive wheels -->
-      <joint_name>front_encoder_wheel_left_joint</joint_name>
-      <joint_name>front_encoder_wheel_right_joint</joint_name>
+      <!--<joint_name>front_encoder_wheel_left_joint</joint_name>
+      <joint_name>front_encoder_wheel_right_joint</joint_name>-->
       <!-- Caster joints -->
       <joint_name>rear_caster_steer_left_joint</joint_name>

File: amr_description/urdf/amr_description.urdf (robot description, URDF)
Before this commit: robot amr_description, 14 links, 13 joints
Joints:
- joint encoder_lift_joint: limit lower=0.01 upper=0.8 effort=50 velocity=0.1 -> lower=0.001 upper=0.8 effort=100 velocity=0.2

Commit message: Octomap

File: amr_description/urdf/amr.gazebo.xacro (robot description, xacro)
@@ -16,5 +16,5 @@
     <parent link="base_footprint"/>
     <child link="base_link"/>
-    <origin xyz="0 0 0.068" rpy="0 0 0"/>
+    <origin xyz="0 0 0.0925" rpy="0 0 0"/>
   </joint>
   <!-- PHYSICAL PROPERTIES -->
@@ -127,13 +127,7 @@
   </gazebo>
   <!-- ============================================================ -->
-  <!-- ASTRA PRO DEPTH CAMERA (RGB + Depth + PointCloud)           -->                       -->
-  <!-- ============================================================ -->
-  <!-- Optical Frame (REP 103 standard) -->
-  <link name="camera_depth_optical_frame"/>
-  <joint name="camera_depth_optical_joint" type="fixed">
-    <parent link="camera_link"/>
-    <child link="camera_depth_optical_frame"/>
-    <origin xyz="0 0 0" rpy="-1.5708 0 -1.5708"/>
-  </joint>
+  <!-- ASTRA PRO DEPTH CAMERA (RGB + Depth + PointCloud)           -->
+  <!-- Optical frame TFs được publish trong launch files (không phải xacro) -->
+  <!-- ============================================================ -->
   <gazebo reference="camera_link">
     <sensor type="depth" name="astra_pro">

Commit message: Change TF

File: amr_description/urdf/amr.gazebo.xacro (robot description, xacro)
@@ -16,5 +16,5 @@
     <parent link="base_footprint"/>
     <child link="base_link"/>
-    <origin xyz="0 0 0.0925" rpy="0 0 0"/>
+    <origin xyz="0 0 0.0926" rpy="0 0 0"/>
   </joint>
   <!-- PHYSICAL PROPERTIES -->

File: amr_description/urdf/amr_description.urdf (robot description, URDF)
Before this commit: robot amr_description, 14 links, 13 joints
Links:
- link base_link: mass 4.3053 -> 4.32441863169069
- link encoder_lift_link: mass 0.8 -> 0.357360840342875
Joints:
- joint base_lift_joint: origin xyz=0.192 0.00019696 0.020997 rpy=0 0 0 -> xyz=0.0511015219283486 0 0.0209015219281041 rpy=0 0 0
- joint camera_joint: origin xyz=0.17 0.0094248 0.59819 rpy=0 0 0 -> xyz=0.0290999999999652 0.00922785541287152 0.598098478071858 rpy=0 0 0
- joint front_encoder_wheel_left_joint: origin xyz=0.1425 0.2361 -0.060003 rpy=0 0 0 -> xyz=0.00160152195240415 0.235903947105134 -0.0600984780718889 rpy=0 0 0
- joint front_encoder_wheel_right_joint: origin xyz=0.1425 -0.2361 -0.060003 rpy=0 0 0 -> xyz=0.00160152195240415 -0.23629785939255 -0.0600984780718906 rpy=0 0 0
- joint left_fork_joint: origin xyz=0.286 0.084803 -0.042399 rpy=0 0 0 -> xyz=0.286001521928153 0.0848030438561962 -0.0423993378150811 rpy=0 0 0
- joint lidar_joint: origin xyz=0.043679 -0.0092089 0.13106 rpy=0 0 0 -> xyz=-0.0972229842064316 -0.00940587864799491 0.130965068568797 rpy=0 0 0
- joint rear_caster_steer_left_joint: origin xyz=-0.1332 0.1931 -0.027503 rpy=0 0 0 -> xyz=-0.274101521928339 0.19290456578464 -0.0275984780718609 rpy=0 0 0
- joint rear_caster_steer_right_joint: origin xyz=-0.1332 -0.1931 -0.027503 rpy=0 0 0 -> xyz=-0.274101521928339 -0.193298478072035 -0.0275984780718622 rpy=0 0 0
- joint rear_caster_wheel_left_joint: origin xyz=0.017 0 -0.0400 rpy=0 0 0 -> xyz=0.0170000000000001 0 -0.0405 rpy=0 0 0
- joint rear_caster_wheel_right_joint: origin xyz=0.017 0 -0.0400 rpy=0 0 0 -> xyz=0.017 0 -0.0405 rpy=0 0 0
- joint right_fork_joint: origin xyz=0.286 -0.085197 -0.042399 rpy=0 0 0 -> xyz=0.28600152192816 -0.0851969561438042 -0.0423993378150817 rpy=0 0 0

Commit message: Fix hardware

File: amr_description/urdf/amr.gazebo.xacro (robot description, xacro)
@@ -16,5 +16,5 @@
     <parent link="base_footprint"/>
     <child link="base_link"/>
-    <origin xyz="0 0 0.0926" rpy="0 0 0"/>
+    <origin xyz="0 0 0.113" rpy="0 0 0"/>
   </joint>
   <!-- PHYSICAL PROPERTIES -->
@@ -175,6 +175,6 @@
       <right_joint>front_encoder_wheel_right_joint</right_joint>
       <!-- Kinematics  -->
-      <wheel_separation>0.4722</wheel_separation>
-      <wheel_diameter>0.065</wheel_diameter>
+      <wheel_separation>0.49</wheel_separation>
+      <wheel_diameter>0.100</wheel_diameter>
       <!-- Limits -->
       <max_wheel_torque>0.863</max_wheel_torque>

File: amr_description/urdf/amr_description.urdf (robot description, URDF)
Before this commit: robot amr_description, 14 links, 13 joints
Links:
- link base_lift_link: mass 0.326486799501112 -> 0.320044401707293
- link base_link: mass 4.32441863169069 -> 4.44724287415331
- link front_encoder_wheel_left_link: mass 0.0241340978121404 -> 0.152554667178822
- link front_encoder_wheel_right_link: mass 0.024134 -> 0.15255466717882
- link left_fork_link: mass 0.0680578875808956 -> 0.0680583578976647
- link rear_caster_steer_left_link: mass 0.0164104146999671 -> 0.0179823003746604
- link rear_caster_steer_right_link: mass 0.017982299786916 -> 0.01798230030437
- link right_fork_link: mass 0.0680578875808746 -> 0.0680583578976465
Joints:
- joint base_lift_joint: origin xyz=0.0511015219283486 0 0.0209015219281041 rpy=0 0 0 -> xyz=0.0495 0.00019696 0.017997 rpy=0 0 0
- joint camera_joint: origin xyz=0.0290999999999652 0.00922785541287152 0.598098478071858 rpy=0 0 0 -> xyz=0.027498 0.0094248 0.59519 rpy=0 0 0
- joint front_encoder_wheel_left_joint: origin xyz=0.00160152195240415 0.235903947105134 -0.0600984780718889 rpy=0 0 0 -> xyz=0 0.2451 -0.063003 rpy=0 0 0
- joint front_encoder_wheel_right_joint: origin xyz=0.00160152195240415 -0.23629785939255 -0.0600984780718906 rpy=0 0 0 -> xyz=0 -0.2451 -0.063003 rpy=0 0 0
- joint left_fork_joint: origin xyz=0.286001521928153 0.0848030438561962 -0.0423993378150811 rpy=0 0 0 -> xyz=0.1275 0.086108 -0.042399 rpy=0 0 0
- joint lidar_joint: origin xyz=-0.0972229842064316 -0.00940587864799491 0.130965068568797 rpy=0 0 0 -> xyz=-0.098654 -0.00075265 0.12981 rpy=0 0 0
- joint rear_caster_steer_left_joint: origin xyz=-0.274101521928339 0.19290456578464 -0.0275984780718609 rpy=0 0 0 -> xyz=-0.2757 0.1931 -0.047753 rpy=0 0 0
- joint rear_caster_steer_right_joint: origin xyz=-0.274101521928339 -0.193298478072035 -0.0275984780718622 rpy=0 0 0 -> xyz=-0.2757 -0.1931 -0.047753 rpy=0 0 0
- joint rear_caster_wheel_left_joint: origin xyz=0.0170000000000001 0 -0.0405 rpy=0 0 0 -> xyz=0.017 0 -0.0405 rpy=0 0 0
- joint right_fork_joint: origin xyz=0.28600152192816 -0.0851969561438042 -0.0423993378150817 rpy=0 0 0 -> xyz=0.1275 -0.085344 -0.042399 rpy=0 0 0
