Commit message: debug hardware

File: amr_description/urdf/amr_description.urdf (robot description, URDF)
Before this commit: robot amr_description, 14 links, 13 joints
Joints:
- joint encoder_lift_joint: limit lower=0.001 upper=0.8 effort=100 velocity=0.2 -> lower=0.0 upper=0.8 effort=100 velocity=0.2

Commit message: Pallet Mission Test

File: amr_description/urdf/amr_description.urdf (robot description, URDF)
Before this commit: robot amr_description, 14 links, 13 joints
Joints:
- joint camera_joint: origin xyz=0.027498 0.0094248 0.59519 rpy=0 0 0 -> xyz=0.027498 0.019688 0.59519 rpy=0.07 0.122 0
